Commit message: all functions of RL working, added also projection in pixel space, orientation of the tool to be fixed

File: Projects/src/doosan-robot/dsr_description/xacro/deburring_tool.urdf.xacro (robot description, xacro)
@@ -33,5 +33,5 @@
 		<parent link="tool" />
 		<child link="tcp" />
-		<origin rpy="-0.17 0 0" xyz="-0.00966 0.00772  0.166" />
+		<origin rpy="0 0 2.46" xyz="-0.00966 0.00772  0.166" />
 	</joint>
   <!-- tcp -->
@@ -52,5 +52,5 @@
 		</visual>
 		<collision>
-			<origin rpy="2.96  0 0" xyz="0 0 0" />
+			<origin rpy="0 0 0" xyz="0 0 0" />
 			<geometry>
 				<sphere radius="0.0015"/>

Commit message: 3Dto2D working. TO DO: use the functions in RL Env

File: Projects/src/doosan-robot/dsr_description/xacro/deburring_tool.urdf.xacro (robot description, xacro)
@@ -5,5 +5,5 @@
 		<inertial>
 			<mass value="0.03"/>
-			<origin rpy="3.14 0 0" xyz="0 0 0" />
+			<origin rpy="0 0 0" xyz="0 0 0" />
 			<inertia ixx="1.76151887e-07" ixy="-3.61499054e-12" ixz="-6.69977864e-11" iyy="1.76154141e-07"
 				iyz="-6.88153918e-11"
@@ -13,11 +13,11 @@
 						<max_contacts>5</max_contacts>
 			<geometry>
-						<mesh filename="package://dsr_description/meshes/gripper/deburring_tool/deburring_tool.stl" scale="1 1 1" />
+						<mesh filename="package://dsr_description/meshes/gripper/deburring_tool/deburring_tool.stl" scale="0.001 0.001 0.001" />
 			</geometry>
 		</collision>
 		<visual>
-						<origin rpy="3.14 0 0" xyz="0 0 0" />
+						<origin rpy="0 0 0" xyz="0 0 0" />
 			<geometry>
-						<mesh filename="package://dsr_description/meshes/gripper/deburring_tool/deburring_tool.stl" scale="1 1 1" />
+						<mesh filename="package://dsr_description/meshes/gripper/deburring_tool/deburring_tool.stl" scale="0.001 0.001 0.001" />
 			</geometry>
 		</visual>
