Commit message: added realsense and sole

File: Projects/src/realsense-ros-gazebo/realsense-ros/realsense2_description/urdf/test_d435i_camera.urdf.xacro (robot description, xacro)
@@ -7,7 +7,13 @@
   <xacro:arg name="add_plug" default="false" />
   <xacro:include filename="$(find realsense2_description)/urdf/_d435i.urdf.xacro"/>
+  <link name="world" />
   <link name="base_link" />
+<joint name="world_joint_camera"  type="fixed">
+    <origin xyz="0.0 0 0.0" rpy="0 0 0" />
+    <parent link="world"/>
+    <child link="base_link"/>
+</joint>
   <xacro:sensor_d435i name="$(arg name)" topics_ns="$(arg topics_ns)" parent="base_link" use_nominal_extrinsics="$(arg use_nominal_extrinsics)" publish_pointcloud="$(arg publish_pointcloud)" add_plug="$(arg add_plug)">
-    <origin xyz="0 0 0" rpy="0 0 0"/>
+    <origin xyz="0 0.5 0.5" rpy="0 1.57 1.57"/>
   </xacro:sensor_d435i>
 </robot>
