Commit message: added package learn to see

File: Projects/src/doosan-robot/sole/description/sole_14.urdf.xacro (robot description, xacro)
@@ -1,15 +1,8 @@
 <?xml version="1.0"?>
 <robot xmlns:xacro="http://www.ros.org/wiki/xacro" name="sole" >
-<!-- sole -->
-<link name="world" />
-<joint name="world_joint"  type="fixed">
-    <origin xyz="0.06 0.7 0.01" rpy="0 0 0" />
-    <parent link="world"/>
-    <child link="sole_link"/>
-</joint>
 <link name="sole_link">
 		<inertial>
 			<mass value="0.3"/>
-			<origin rpy="1.57 -3.14 0 " xyz="0 0 0" />
+			<origin rpy="0 0 0 " xyz="0.0 0.0 0.0" />
 			<inertia ixx="0" ixy="0" ixz="0" iyy="0"
 				iyz="0"
@@ -19,16 +12,22 @@
 						<max_contacts>5</max_contacts>
 			<geometry>
-						<mesh filename="package://sole/meshes/sole.stl" scale="1 1 1" />
+						<mesh filename="package://sole/meshes/sole_14.stl" scale="0.001 0.001 0.001" />
 			</geometry>
 		</collision>
 		<visual>
-			            <origin rpy="1.57 -3.14 0 " xyz="0 0 0 " />
+			            <origin rpy=" 0 0 0 " xyz="0 0 0" />
 			<geometry>
-						<mesh filename="package://sole/meshes/sole.stl" scale="1 1 1" />
+						<mesh filename="package://sole/meshes/sole_14.stl" scale="0.001 0.001 0.001" />
 			</geometry>
 		</visual>
+		<gazebo>
+			<static>true</static>
+		</gazebo>
 	</link>
   <gazebo reference="sole_link">
     <material>Gazebo/Black</material>
   </gazebo>
+<gazebo>
+    <static>true</static>
+</gazebo>
 </robot>
